File: MacroPad.kicad_pcb (KiCad board)
At the start: 2 copper layers, 105 x 131 mm, 46 parts, among them SW1 SW_Push, SW10 SW_Push, SW11 SW_Push, SW12 SW_Push, SW13 SW_Push, SW14 SW_Push, SW15 SW_Push, SW16 SW_Push, SW17 SW_Push, SW18 SW_Push, SW19 SW_Push, SW2 SW_Push, SW20 SW_Push, SW21 SW_Push, SW22 SW_Push, SW3 SW_Push, SW4 SW_Push, SW5 SW_Push, SW6 SW_Push, SW7 SW_Push, SW8 SW_Push, SW9 SW_Push

Commit message: wheee
Parts:
- added REF**: MountingHole_2.2mm_M2, MountingHole:MountingHole_2.2mm_M2, F.Cu at (145.0, 46.0)
- added REF**: MountingHole_2.2mm_M2, MountingHole:MountingHole_2.2mm_M2, F.Cu at (145.0, 167.0)
- added REF**: MountingHole_2.2mm_M2, MountingHole:MountingHole_2.2mm_M2, F.Cu at (50.0, 46.0)
- added REF**: MountingHole_2.2mm_M2, MountingHole:MountingHole_2.2mm_M2, F.Cu at (50.0, 167.0)
- added SWR: SW_Push_1P1T_XKB_TS-1187A, Button_Switch_SMD:SW_Push_1P1T_XKB_TS-1187A, B.Cu at (97.5, 50.0)
- D1, D10, D11, D12, D13, D14, D15, D16, D17, D18, D19, D2, D20, D21, D22, D3, D4, D5, D6, D7, D8, D9: footprint D_SOD-123 -> sea-picro:D_SOD-123-Stripe
- moved REF** 1.17 mm to (61.6, 58.1)
Routing:
- net ROW4: track 74.6 -> 198.7 mm, vias 0 -> 8
- net ROW3: track 78.9 -> 172.1 mm, vias 0 -> 8
- net ROW2: track 84.1 -> 155.7 mm, vias 0 -> 2
- net COL4: track 87.4 -> 149.8 mm
- net RST: track 0.00 -> 58.4 mm
- net ROW1: track 78.8 -> 129.7 mm, vias 0 -> 2
- net COL3: track 73.7 -> 119.3 mm
- net COL2: track 87.9 -> 117.4 mm
- net ROW0: track 76.2 -> 102.7 mm
- net COL1: track 99.7 -> 116.7 mm
- net COL0: track 57.2 -> 73.0 mm
- net GND: vias 0 -> 13
- added copper zone on B.Cu, net GND
- added copper zone on F.Cu, net GND
