File: MacroPad.kicad_pcb (KiCad board)
At the start: 2 copper layers, 105 x 131 mm, 51 parts, among them SW1 SW_Push, SW10 SW_Push, SW11 SW_Push, SW12 SW_Push, SW13 SW_Push, SW14 SW_Push, SW15 SW_Push, SW16 SW_Push, SW17 SW_Push, SW18 SW_Push, SW19 SW_Push, SW2 SW_Push, SW20 SW_Push, SW21 SW_Push, SW22 SW_Push, SW3 SW_Push, SW4 SW_Push, SW5 SW_Push, SW6 SW_Push, SW7 SW_Push, SW8 SW_Push, SW9 SW_Push

Commit message: switch mcu to pico
Parts:
- removed the REF** at (61.6, 58.1)
- added REF**: RaspberryPi_Pico_Common_THT, Module:RaspberryPi_Pico_Common_THT, F.Cu at (47.4, 69.2)
- moved SWR 17.5 mm to (115.0, 50.0)
Routing:
- net ROW4: track 198.7 -> 177.8 mm
- net COL2: track 117.4 -> 138.2 mm
- net ROW3: track 172.1 -> 155.6 mm, vias 8 -> 7
- net ROW2: track 155.7 -> 141.9 mm, vias 2 -> 3
- net COL1: track 116.7 -> 127.0 mm
- net ROW1: track 129.7 -> 120.5 mm, vias 2 -> 3
- net COL4: track 149.8 -> 158.4 mm
- net COL3: track 119.3 -> 127.9 mm
- net ROW0: track 102.7 -> 96.2 mm
- net COL0: track 73.0 -> 68.6 mm
