File: MacroPad.kicad_pcb (KiCad board)
At the start: 2 copper layers, 105 x 131 mm, 51 parts, among them SW1 SW_Push, SW10 SW_Push, SW11 SW_Push, SW12 SW_Push, SW13 SW_Push, SW14 SW_Push, SW15 SW_Push, SW16 SW_Push, SW17 SW_Push, SW18 SW_Push, SW19 SW_Push, SW2 SW_Push, SW20 SW_Push, SW21 SW_Push, SW22 SW_Push, SW3 SW_Push, SW4 SW_Push, SW5 SW_Push, SW6 SW_Push, SW7 SW_Push, SW8 SW_Push, SW9 SW_Push

Commit message: update pcb
Parts:
- moved REF** 1.03 mm to (48.4, 69.2)
Routing:
- net COL2: track 138.2 -> 127.1 mm
- net RST: track 58.4 -> 50.2 mm
- net COL4: track 158.4 -> 157.2 mm
- net ROW4: track 177.8 -> 177.0 mm
- net COL3: track 127.9 -> 127.1 mm
- net ROW0: track 96.2 -> 96.8 mm
